File: ASIC.kicad_sch (KiCad schematic)
At the start: 77 parts, among them U10 BM1370_mode1, U11 MCP1824T-1202E/OT, U12 MCP1824T-0802E, U2 SN74AVC4T774, U8 25MHz, U9 BM1370_mode1

Commit message: ASIC.sch update in BM footprint
Parts:
- U10, U9: footprint bitaxe:BM1370 -> bitaxe:BM1370_JB
Changed lines of the file:
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@@
 			)
 		)
-		(property "Footprint" "bitaxe:BM1370"
+		(property "Footprint" "bitaxe:BM1370_JB"
 			(at 115.57 147.32 0)
 			(effects
@@
 			)
 		)
-		(property "Footprint" "bitaxe:BM1370"
+		(property "Footprint" "bitaxe:BM1370_JB"
 			(at 219.71 147.32 0)
 			(effects
